Commit message: try to fix the controllers

File: rover_description/urdf/arm/arm.urdf.xacro (robot description, xacro)
@@ -13,5 +13,5 @@
     </joint>
     <joint name="Brazo_L3_link_joint" type="prismatic">
-      <limit lower="0.00000" upper="1.70000" effort="50.0" velocity="1.5"/>
+      <limit lower="0.00000" upper="1.70000" effort="100" velocity="100.0"/>
       <origin rpy="0.00000 0.00000 1.57080" xyz="0.00000 0.00000 -1.00000"/>
       <parent link="Union_L2_L3_link"/>
@@ -40,5 +40,5 @@
     </joint>
     <joint name="Union_base_L1_link_joint" type="revolute">
-      <limit lower="-2.50000" upper="2.50000" effort="50.0" velocity="1.5"/>
+      <limit lower="-2.50000" upper="2.50000" effort="100" velocity="100.0"/>
       <origin rpy="0.00000 0.00000 1.57080" xyz="0.00000 0.00000 1.00000"/>
       <parent link="Brazo_base_link"/>
@@ -47,5 +47,5 @@
     </joint>
     <joint name="Union_eje_L2_link_joint" type="revolute">
-      <limit lower="-2.50000" upper="2.50000" effort="50.0" velocity="1.5"/>
+      <limit lower="-2.50000" upper="2.50000" effort="100" velocity="100.0"/>
       <origin rpy="0.00000 0.00000 1.57080" xyz="0.00000 0.00000 -0.25000"/>
       <parent link="Union_L1_L2_link"/>

File: rover_description/urdf/arm/gripper.urdf.xacro (robot description, xacro)
@@ -3,5 +3,5 @@
   <xacro:macro name="gripper" params="parent">
     <joint name="Base_pinza_link_joint" type="continuous">
-      <limit effort="50.0" velocity="1.5"/>
+      <limit effort="100.0" velocity="100"/>
       <origin rpy="3.1416 0.00000 -1.57080" xyz="0.00000 0.00000 -1.00000"/>
       <parent link="${parent}"/>
@@ -10,5 +10,5 @@
     </joint>
     <joint name="Dedo_der_link_joint" type="prismatic">
-      <limit lower="0.00000" upper="0.45000" effort="50.0" velocity="1.5"/>
+      <limit lower="0.00000" upper="0.45000" effort="100" velocity="100.0"/>
       <origin rpy="0.00000 0.00000 3.1416" xyz="0.57500 0.00000 0.17500"/>
       <parent link="Base_pinza_link"/>
@@ -17,5 +17,5 @@
     </joint>
     <joint name="Dedo_iz_link_joint" type="prismatic">
-      <limit lower="0.00000" upper="0.45000" effort="50.0" velocity="1.5"/>
+      <limit lower="0.00000" upper="0.45000" effort="100" velocity="100.0"/>
       <origin rpy="0.00000 0.00000 0.00000" xyz="-0.57500 0.00000 0.17500"/>
       <parent link="Base_pinza_link"/>
